Commit message: finish the dexter version of description and moveit_config, can run the launch.demo

File: src/dexter_description/urdf_dexter/robot.urdf (robot description, URDF)
Before this commit: robot dexter_simplify, 7 links, 6 joints
Links:
- added link tool_link
Joints:
- added joint hand_tool_joint: type fixed, parent part6, child tool_link, origin xyz=0 0 -0.03 rpy=3.14159 0 0
