Commit message: finish the JTC connect to real hardware, but have work yet

File: src/dexter_moveit_config/config/dexter_simplify.ros2_control.xacro (robot description, xacro)
@@ -1,10 +1,35 @@
 <?xml version="1.0"?>
 <robot xmlns:xacro="http://www.ros.org/wiki/xacro">
-    <xacro:macro name="dexter_simplify_ros2_control" params="name initial_positions_file">
+    <xacro:macro name="dexter_simplify_ros2_control" params="
+        name initial_positions_file use_hardware can_interface can_bitrate encoder_timeout_us
+        max_speed_field min_speed_field fallback_speed_field acceleration_field
+        velocity_filter_alpha max_command_step_rad">
         <xacro:property name="initial_positions" value="${xacro.load_yaml(initial_positions_file)['initial_positions']}"/>
         <ros2_control name="${name}" type="system">
             <hardware>
-                <!-- By default, set up controllers for simulation. This won't work on real hardware -->
-                <plugin>mock_components/GenericSystem</plugin>
+                <xacro:if value="${use_hardware}">
+                    <plugin>dexter_hardware/DexterSystem</plugin>
+                    <param name="can_interface">${can_interface}</param>
+                    <param name="can_bitrate">${can_bitrate}</param>
+                    <param name="encoder_timeout_us">${encoder_timeout_us}</param>
+                    <param name="startup_quiet_period_us">20000</param>
+                    <param name="startup_max_wait_us">250000</param>
+                    <param name="max_speed_field">${max_speed_field}</param>
+                    <param name="min_speed_field">${min_speed_field}</param>
+                    <param name="fallback_speed_field">${fallback_speed_field}</param>
+                    <param name="acceleration_field">${acceleration_field}</param>
+                    <param name="part5_min_speed_field">1</param>
+                    <param name="part5_fallback_speed_field">1</param>
+                    <param name="part5_acceleration_field">0</param>
+                    <param name="velocity_filter_alpha">${velocity_filter_alpha}</param>
+                    <param name="max_command_step_rad">${max_command_step_rad}</param>
+                    <param name="configure_part5_driver">true</param>
+                    <param name="part5_work_mode">4</param>
+                    <param name="part5_working_current_ma">800</param>
+                    <param name="part5_subdivisions">128</param>
+                </xacro:if>
+                <xacro:unless value="${use_hardware}">
+                    <plugin>mock_components/GenericSystem</plugin>
+                </xacro:unless>
             </hardware>
             <joint name="base">

File: src/dexter_moveit_config/config/dexter_simplify.urdf.xacro (robot description, xacro)
@@ -2,8 +2,30 @@
 <robot xmlns:xacro="http://www.ros.org/wiki/xacro" name="dexter_simplify">
     <xacro:arg name="initial_positions_file" default="initial_positions.yaml" />
+    <xacro:arg name="use_hardware" default="false" />
+    <xacro:arg name="can_interface" default="can0" />
+    <xacro:arg name="can_bitrate" default="1000000" />
+    <xacro:arg name="encoder_timeout_us" default="2000" />
+    <xacro:arg name="max_speed_field" default="3000" />
+    <xacro:arg name="min_speed_field" default="10" />
+    <xacro:arg name="fallback_speed_field" default="300" />
+    <xacro:arg name="acceleration_field" default="0" />
+    <xacro:arg name="velocity_filter_alpha" default="0.25" />
+    <xacro:arg name="max_command_step_rad" default="0.05" />
     <!-- Import the current Dexter model and its collision geometry. -->
     <xacro:include filename="$(find dexter_description)/fix_with_limit/robot.urdf" />
     <!-- Import control_xacro -->
     <xacro:include filename="dexter_simplify.ros2_control.xacro" />
-    <xacro:dexter_simplify_ros2_control name="FakeSystem" initial_positions_file="$(arg initial_positions_file)"/>
+    <xacro:dexter_simplify_ros2_control
+        name="DexterSystem"
+        initial_positions_file="$(arg initial_positions_file)"
+        use_hardware="$(arg use_hardware)"
+        can_interface="$(arg can_interface)"
+        can_bitrate="$(arg can_bitrate)"
+        encoder_timeout_us="$(arg encoder_timeout_us)"
+        max_speed_field="$(arg max_speed_field)"
+        min_speed_field="$(arg min_speed_field)"
+        fallback_speed_field="$(arg fallback_speed_field)"
+        acceleration_field="$(arg acceleration_field)"
+        velocity_filter_alpha="$(arg velocity_filter_alpha)"
+        max_command_step_rad="$(arg max_command_step_rad)"/>
 </robot>
