Commit message: before the urdf change

File: src/dexter_description/base/robot.urdf (robot description, URDF)
Before this commit: robot dexter_simplify, 8 links, 7 joints
Links:
- removed link gripper_tip
- link base: geometry collision mesh filename=package://assets/base.stl; visual mesh filename=package://assets/base.stl
- link part1: geometry collision mesh filename=package://assets/part1.stl; visual mesh filename=package://assets/part1.stl
- link part2: geometry collision mesh filename=package://assets/part2.stl; visual mesh filename=package://assets/part2.stl
- link part3: geometry collision mesh filename=package://assets/part3.stl; visual mesh filename=package://assets/part3.stl
- link part4: geometry collision mesh filename=package://assets/part4.stl; visual mesh filename=package://assets/part4.stl
- link part5: geometry collision mesh filename=package://assets/part5.stl; visual mesh filename=package://assets/part5.stl
- link part6: geometry collision mesh filename=package://assets/part6.stl; visual mesh filename=package://assets/part6.stl
Joints:
- removed joint gripper_tip_joint
- joint base: limit lower=-2.2689280275926285 upper=2.2689280275926285 effort=10 velocity=10 -> lower=-3.141592653589793 upper=3.141592653589793 effort=10 velocity=10; origin xyz=-2.91434e-16 -7.91034e-16 0.1085 rpy=3.14159 -0 -5.55112e-16 -> xyz=0 0 0.1085 rpy=3.14159 -0 0
- joint part1: limit lower=-1.2217304763960306 upper=1.5707963267948966 effort=10 velocity=10 -> lower=-1.5708 upper=1.5708 effort=10 velocity=10; origin xyz=-4.85723e-18 0.04 -0.032057 rpy=-1.5708 -4.33876e-25 3.14159 -> xyz=-1.04083e-17 0.04 -0.032057 rpy=-1.5708 -1.10203e-38 3.14159
- joint part2: origin xyz=-8.27116e-17 0.102 0.0615 rpy=-3.14159 -7.77156e-16 -1.5708 -> xyz=-4.85723e-17 0.102 0.0615 rpy=-3.14159 -7.77156e-16 -1.5708
- joint part3: limit lower=-1.7453292519943295 upper=1.7453292519943295 effort=10 velocity=10 -> lower=-3.141592653589793 upper=3.141592653589793 effort=10 velocity=10
- joint part4: origin xyz=-5.55112e-17 -0.029 -0.057529 rpy=-1.5708 -1.5708 0 -> xyz=-1.11022e-16 -0.029 -0.057529 rpy=-1.5708 -1.5708 0
- joint part5: limit lower=-6.1959188446 upper=0.0872665 effort=10 velocity=10 -> lower=-3.141592653589793 upper=3.141592653589793 effort=10 velocity=10; origin xyz=0 -0.062 0.028 rpy=-1.5708 1.5708 0 -> xyz=-1.38778e-17 -0.062 0.028 rpy=-1.5708 1.5708 0
