Commit message: correct gripper tip position

File: src/dexter_description/fix_with_limit/robot.urdf (robot description, URDF)
Before this commit: robot dexter_simplify, 8 links, 7 joints
Joints:
- joint gripper_tip_joint: origin xyz=0 0.085 0.0285 rpy=-1.5708 0 0 -> xyz=0 0.073 -0.035 rpy=1.5708 3.14159 0

Commit message: change the URDF joint limit, set part5 to 800mA

File: src/dexter_description/fix_with_limit/robot.urdf (robot description, URDF)
Before this commit: robot dexter_simplify, 8 links, 7 joints
Joints:
- joint base: limit lower=-3.141592653589793 upper=3.141592653589793 effort=10 velocity=10 -> lower=-2.2689280275926285 upper=2.2689280275926285 effort=10 velocity=10
- joint part1: limit lower=-1.5708 upper=1.5708 effort=10 velocity=10 -> lower=-1.2217304763960306 upper=1.5707963267948966 effort=10 velocity=10
- joint part3: limit lower=-3.141592653589793 upper=3.141592653589793 effort=10 velocity=10 -> lower=-1.7453292519943295 upper=1.7453292519943295 effort=10 velocity=10

Commit message: urdf file changed

File: src/dexter_description/fix_with_limit/robot.urdf (robot description, URDF)
Before this commit: robot dexter_simplify, 8 links, 7 joints
Joints:
- joint base: origin xyz=-2.91434e-16 -7.91034e-16 0.1085 rpy=3.14159 -0 -5.55112e-16 -> xyz=0 0 0.1085 rpy=3.14159 -0 0
